File: arisu.kicad_pcb (KiCad board)
At the start: 2 copper layers, 339.1 x 118.7 mm, 176 parts, among them J1 USB_B_Micro, SW1 SW_Push, SW10 SW_Push, SW11 SW_Push, SW12 SW_Push, SW13 SW_Push, SW14 SW_Push, SW15 SW_Push, SW16 SW_Push, SW17 SW_Push, SW18 SW_Push, SW19 SW_Push, SW2 SW_Push, SW20 SW_Push, SW21 SW_Push, SW22 SW_Push, SW23 SW_Push, SW24 SW_Push, SW25 SW_Push, SW26 SW_Push, SW27 SW_Push, SW28 SW_Push, SW29 SW_Push, SW3 SW_Push, SW30 SW_Push, SW31 SW_Push, SW32 SW_Push, SW33 SW_Push, SW34 SW_Push, SW35 SW_Push, SW36 SW_Push, SW37 SW_Push, SW38 SW_Push, SW39 SW_Push, SW4 SW_Push, SW40 SW_Push, SW41 SW_Push, SW42 SW_Push, SW43 SW_Push, SW44 SW_Push, SW45 SW_Push, SW46 SW_Push, SW47 SW_Push, SW48 SW_Push, SW49 SW_Push, SW5 SW_Push, SW50 SW_Push, SW51 SW_Push, SW52 SW_Push, SW53 SW_Push, SW54 SW_Push, SW55 SW_Push, SW56 SW_Push, SW57 SW_Push, SW58 SW_Push, SW59 SW_Push, SW6 SW_Push, SW60 SW_Push, SW61 SW_Push, SW62 SW_Push, SW63 SW_Push, SW64 SW_Push, SW65 SW_Push, SW66 SW_Push, SW67 SW_Push, SW7 SW_Push, SW8 SW_Push, SW9 SW_Push, U1 USBLC6-2SC6, U2 ATmega32U4-AU, Y1 Crystal_GND24

Commit message: Add hotswap and USB-C
Add hotswap and USB-C
Parts:
- removed D+: D+, Pin_Headers:Pin_Header_Straight_1x01_Pitch2.54mm
- removed D-: D-, Pin_Headers:Pin_Header_Straight_1x01_Pitch2.54mm
- removed G*** (x2): LOGO, arisu:arisu-logo
- removed GND: GND, Pin_Headers:Pin_Header_Straight_1x01_Pitch2.54mm
- removed VCC: VCC, Pin_Headers:Pin_Header_Straight_1x01_Pitch2.54mm
- added F1: 500mA, Fuse:Fuse_1206_3216Metric_Pad1.42x1.75mm_HandSolder, B.Cu at (171.2, 31.6)
- added J12: D+, Connector_PinHeader_2.54mm:PinHeader_1x01_P2.54mm_Vertical, B.Cu at (143.8, 26.4)
- added J13: D-, Connector_PinHeader_2.54mm:PinHeader_1x01_P2.54mm_Vertical, B.Cu at (146.3, 26.4)
- added J14: GND, Connector_PinHeader_2.54mm:PinHeader_1x01_P2.54mm_Vertical, B.Cu at (148.9, 26.4)
- added R5: 5.1k, Resistor_SMD:R_0805_2012Metric_Pad1.20x1.40mm_HandSolder, B.Cu at (188.1, 28.7)
- added R6: 5.1k, Resistor_SMD:R_0805_2012Metric_Pad1.20x1.40mm_HandSolder, B.Cu at (186.0, 26.2)
- added USB1: HRO-TYPE-C-31-M-12, Type-C:HRO-TYPE-C-31-M-12-HandSoldering, B.Cu at (175.4, 19.0)
- D1, D10, D11, D12, D13, D14, D15, D16, D17, D18, D19, D2, D20, D21, D22, D23, D24, D25, D26, D27, D28, D29, D3, D30, D31, D32, D33, D34, D35, D36, D37, D38, D39, D4, D40, D41, D42, D43, D44, D45, D46, D47, D48, D49, D5, D50, D51, D52, D53, D54, D55, D56, D57, D58, D59, D6, D60, D61, D62, D63, D64, D65, D66, D67, D7, D8, D9: footprint Diodes_SMD:D_SOD-123 -> Diode_SMD:D_SOD-123
- J1: value USB_B_Micro -> VCC; footprint Connectors_USB:USB_Micro-B_Molex-105017-0001 -> Connector_PinHeader_2.54mm:PinHeader_1x01_P2.54mm_Vertical
- J10: renamed from PF6; footprint Pin_Headers:Pin_Header_Straight_1x01_Pitch2.54mm -> Connector_PinHeader_2.54mm:PinHeader_1x01_P2.54mm_Vertical
- J11: renamed from PF7; footprint Pin_Headers:Pin_Header_Straight_1x01_Pitch2.54mm -> Connector_PinHeader_2.54mm:PinHeader_1x01_P2.54mm_Vertical
- J2: renamed from MISO; footprint Pin_Headers:Pin_Header_Straight_1x01_Pitch2.54mm -> Connector_PinHeader_2.54mm:PinHeader_1x01_P2.54mm_Vertical
- J3: renamed from VCC; footprint Pin_Headers:Pin_Header_Straight_1x01_Pitch2.54mm -> Connector_PinHeader_2.54mm:PinHeader_1x01_P2.54mm_Vertical
- J4: renamed from SCK; footprint Pin_Headers:Pin_Header_Straight_1x01_Pitch2.54mm -> Connector_PinHeader_2.54mm:PinHeader_1x01_P2.54mm_Vertical
- J5: renamed from MOSI; footprint Pin_Headers:Pin_Header_Straight_1x01_Pitch2.54mm -> Connector_PinHeader_2.54mm:PinHeader_1x01_P2.54mm_Vertical
- J6: renamed from RES; footprint Pin_Headers:Pin_Header_Straight_1x01_Pitch2.54mm -> Connector_PinHeader_2.54mm:PinHeader_1x01_P2.54mm_Vertical
- J7: renamed from GND; footprint Pin_Headers:Pin_Header_Straight_1x01_Pitch2.54mm -> Connector_PinHeader_2.54mm:PinHeader_1x01_P2.54mm_Vertical
- J8: renamed from PF4; footprint Pin_Headers:Pin_Header_Straight_1x01_Pitch2.54mm -> Connector_PinHeader_2.54mm:PinHeader_1x01_P2.54mm_Vertical
- J9: renamed from PF5; footprint Pin_Headers:Pin_Header_Straight_1x01_Pitch2.54mm -> Connector_PinHeader_2.54mm:PinHeader_1x01_P2.54mm_Vertical
- R1, R2, R3, R4: footprint Resistors_SMD:R_0805_HandSoldering -> Resistor_SMD:R_0805_2012Metric_Pad1.20x1.40mm_HandSolder
- SW1, SW10, SW11, SW12, SW13, SW15, SW16, SW17, SW18, SW19, SW20, SW21, SW22, SW24, SW25, SW26, SW27, SW28, SW29, SW30, SW31, SW32, SW33, SW34, SW35, SW36, SW38, SW39, SW40, SW41, SW42, SW43, SW44, SW45, SW47, SW48, SW49, SW50, SW51, SW52, SW53, SW55, SW56, SW58, SW59, SW6, SW61, SW62, SW63, SW64, SW65, SW66, SW67, SW7, SW8, SW9: footprint MX_Switch:SW_Cherry_MX_1.00u_PCB -> MX_Only:MXOnly-1U-Hotswap
- SW14, SW2, SW46, SW5, SW60: footprint MX_Switch:SW_Cherry_MX_1.50u_PCB -> MX_Only:MXOnly-1.5U-Hotswap
- SW23: footprint MX_Switch:SW_Cherry_MX_2.00u_PCB_ReversedStabilizers -> MX_Only:MXOnly-2U-Hotswap-ReversedStabilizers
- SW3, SW54: footprint MX_Switch:SW_Cherry_MX_1.75u_PCB -> MX_Only:MXOnly-1.75U-Hotswap
- SW37: footprint MX_Switch:SW_Cherry_MX_2.75u_PCB_ReversedStabilizers -> MX_Only:MXOnly-2.75U-Hotswap-ReversedStabilizers
- SW4: footprint MX_Switch:SW_Cherry_MX_2.25u_PCB -> MX_Only:MXOnly-2.25U-Hotswap
- SW57: footprint MX_Switch:SW_Cherry_MX_2.25u_PCB_ReversedStabilizers -> MX_Only:MXOnly-2.25U-Hotswap-ReversedStabilizers
- U1: value USBLC6-2SC6 -> SRV05-4; footprint TO_SOT_Packages_SMD:SOT-23-6_Handsoldering -> Package_TO_SOT_SMD:SOT-23-6
- moved SW37 27.9 mm to (212.4, 126.4)
- moved J1 24.1 mm to (151.4, 26.4)
- moved SW4 23.5 mm to (46.9, 95.8)
- moved SW57 23.5 mm to (319.3, 76.8)
- moved SW23 21.3 mm to (131.6, 124.9)
- moved SW54 19.2 mm to (305.0, 95.9)
- moved SW3 19.2 mm to (46.2, 76.8)
- moved SW46 17.2 mm to (252.0, 118.0)
- moved SW2 17.2 mm to (48.0, 57.8)
- moved SW5 17.2 mm to (39.7, 114.9)
- moved SW60 17.2 mm to (322.1, 57.8)
- moved SW14 17.2 mm to (99.0, 117.9)
- moved SW64 13.5 mm to (346.6, 34.0)
- moved SW30 13.5 mm to (184.2, 74.0)
- moved SW39 13.5 mm to (221.5, 66.0)
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Connections:
- R1 pad 1: D+ -> Net-(J13-Pad1)
- R1 pad 2: Net-(J1-Pad3) -> D-
- R2 pad 1: D- -> D+
- R2 pad 2: Net-(J1-Pad2) -> Net-(J12-Pad1)
- U1 pad 1: Net-(U1-Pad1) -> Net-(J13-Pad1)
- U1 pad 4: Net-(J1-Pad2) -> Net-(U1-Pad4)
- U1 pad 6: Net-(J1-Pad3) -> Net-(J12-Pad1)
Routing:
- net /row4: track 433.8 -> 580.3 mm, vias 2 -> 4
- net Net-(J12-Pad1): track 0.00 -> 49.3 mm, vias 0 -> 2
- net Net-(J1-Pad3): track 47.8 -> 0.00 mm
- net Net-(J1-Pad2): track 45.1 -> 0.00 mm
- net GND: track 71.6 -> 111.8 mm, vias 12 -> 15
- net Net-(J13-Pad1): track 0.00 -> 38.2 mm, vias 0 -> 2
- net /col5: track 121.5 -> 158.2 mm, vias 0 -> 7
- net /col4: track 135.2 -> 171.0 mm, vias 0 -> 7
- net /col10: track 221.3 -> 188.7 mm, vias 0 -> 5
- net /SCK: track 157.0 -> 182.7 mm, vias 2 -> 7
- net /col2: track 175.7 -> 199.9 mm, vias 2 -> 9
- net /col0: track 204.4 -> 228.2 mm, vias 0 -> 5
- net /col3: track 133.3 -> 153.8 mm, vias 0 -> 4
- net /col6: track 96.8 -> 116.9 mm, vias 0 -> 4
- net /col1: track 166.8 -> 185.8 mm, vias 0 -> 4
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Other:
- board size 339.1 x 118.7 mm -> 339.1 x 124.1 mm

Commit message: Update footprints
Update backspace to 2U, left spacebar to 2.25U, left Alt to 1.25U
Parts:
- removed the D63 at (331.0, 40.5)
- removed the SW63 at (322.7, 38.7)
- SW14: footprint MX_Only:MXOnly-1.5U-Hotswap -> MX_Only:MXOnly-1.25U-Hotswap
- SW23: footprint MX_Only:MXOnly-2U-Hotswap-ReversedStabilizers -> MX_Only:MXOnly-2.25U-Hotswap-ReversedStabilizers
- SW59: footprint MX_Only:MXOnly-1U-Hotswap -> MX_Only:MXOnly-2U-Hotswap
- moved SW59 9.53 mm to (313.2, 38.7)
- moved D59 9.52 mm to (321.5, 40.5)
- moved C7 3.73 mm to (179.3, 53.2), turned to 270 degrees
- moved H7 2.86 mm to (338.9, 45.2)
- moved SW14 2.37 mm to (96.7, 117.5)
- moved SW23 2.30 mm to (129.3, 124.4)
- moved D14 1.93 mm to (104.0, 121.4)
- renumbered D64 to D63, D65 to D64, D66 to D65, D67 to D66, J2 to J1, J14 to J10, J8 to J11, J9 to J12, J10 to J13, J11 to J14, J3 to J2, J4 to J3, J5 to J4, J6 to J5, J7 to J6, J1 to J7, J12 to J8, J13 to J9, R5 to R1, R6 to R2, R1 to R3, R2 to R4, R3 to R5, R4 to R6, SW64 to SW63, SW65 to SW64, SW66 to SW65, SW67 to SW66
Connections:
- C3 pad 1: VCC -> +5V
- C5 pad 1: VCC -> +5V
- C6 pad 1: VCC -> +5V
- C7 pad 1: VCC -> +5V
- C8 pad 1: VCC -> +5V
- C9 pad 1: VCC -> +5V
- F1 pad 1: VCC -> +5V
- J2 pad 1: VCC -> +5V
- R5 pad 1: VCC -> +5V
- U1 pad 5: VCC -> +5V
- U2 pad 14: VCC -> +5V
- U2 pad 2: VCC -> +5V
- U2 pad 24: VCC -> +5V
- U2 pad 34: VCC -> +5V
- U2 pad 44: VCC -> +5V
- U2 pad 7: VCC -> +5V
Routing:
- net +5V: track 0.00 -> 187.2 mm, vias 0 -> 7
- net VCC: track 208.8 -> 34.2 mm, vias 11 -> 3
- net /col5: track 158.2 -> 141.4 mm, vias 7 -> 5
- net /col4: track 171.0 -> 159.3 mm, vias 7 -> 5
- net /row0: track 331.5 -> 321.2 mm
- net Net-(D63-Pad2) (its old number): track 6.21 -> 0.00 mm
- net /col12: track 236.5 -> 230.3 mm, vias 7 -> 5
- net /col2: track 199.9 -> 196.6 mm
- net /MISO: track 273.9 -> 270.6 mm
- net /row4: track 580.3 -> 583.0 mm
- net GND: track 111.8 -> 109.9 mm, vias 15 -> 16
- net Net-(D23-Pad2): track 6.20 -> 7.64 mm
- net /col6: track 116.9 -> 118.0 mm, vias 4 -> 6
- net Net-(D14-Pad2): track 7.33 -> 6.49 mm
- net /col10: track 188.7 -> 189.5 mm
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Other:
- board text removed: "Fate Design Rev 1.1"

Commit message: RGB in Progress
RGB in Progress
Parts:
- removed J14: PF7, Connector_PinHeader_2.54mm:PinHeader_1x01_P2.54mm_Vertical
- added C10: 0.1uF, Capacitor_SMD:C_0805_2012Metric_Pad1.18x1.45mm_HandSolder, B.Cu at (144.2, 31.4)
- added C11: 0.1uF, Capacitor_SMD:C_0805_2012Metric_Pad1.18x1.45mm_HandSolder, B.Cu at (69.8, 27.8)
- added C12: 0.1uF, Capacitor_SMD:C_0805_2012Metric_Pad1.18x1.45mm_HandSolder, B.Cu at (32.5, 48.4)
- added C13: 0.1uF, Capacitor_SMD:C_0805_2012Metric_Pad1.18x1.45mm_HandSolder, B.Cu at (32.3, 80.2)
- added C14: 0.1uF, Capacitor_SMD:C_0805_2012Metric_Pad1.18x1.45mm_HandSolder, B.Cu at (30.3, 126.0)
- added C15: 0.1uF, Capacitor_SMD:C_0805_2012Metric_Pad1.18x1.45mm_HandSolder, B.Cu at (74.6, 123.8)
- added C16: 0.1uF, Capacitor_SMD:C_0805_2012Metric_Pad1.18x1.45mm_HandSolder, B.Cu at (183.1, 138.9)
- added C17: 0.1uF, Capacitor_SMD:C_0805_2012Metric_Pad1.18x1.45mm_HandSolder, B.Cu at (275.6, 152.9)
- added C18: 0.1uF, Capacitor_SMD:C_0805_2012Metric_Pad1.18x1.45mm_HandSolder, B.Cu at (349.8, 150.3)
- added C19: 0.1uF, Capacitor_SMD:C_0805_2012Metric_Pad1.18x1.45mm_HandSolder, B.Cu at (385.6, 112.1)
- added C20: 0.1uF, Capacitor_SMD:C_0805_2012Metric_Pad1.18x1.45mm_HandSolder, B.Cu at (385.9, 58.5)
- added C21: 0.1uF, Capacitor_SMD:C_0805_2012Metric_Pad1.18x1.45mm_HandSolder, B.Cu at (366.9, 8.12)
- added C22: 0.1uF, Capacitor_SMD:C_0805_2012Metric_Pad1.18x1.45mm_HandSolder, B.Cu at (309.8, 0.98)
- added C23: 0.1uF, Capacitor_SMD:C_0805_2012Metric_Pad1.18x1.45mm_HandSolder, B.Cu at (227.5, 0.36)
- added R7: 510, Resistor_SMD:R_0805_2012Metric_Pad1.20x1.40mm_HandSolder, B.Cu at (136.1, 32.3)
- added RGB1: WS2812B, LED_SMD:LED_WS2812B_PLCC4_5.0x5.0mm_P3.2mm, B.Cu at (130.1, 29.5)
- added RGB10: WS2812B, LED_SMD:LED_WS2812B_PLCC4_5.0x5.0mm_P3.2mm, B.Cu at (353.1, 7.44)
- added RGB11: WS2812B, LED_SMD:LED_WS2812B_PLCC4_5.0x5.0mm_P3.2mm, B.Cu at (69.8, 123.8)
- added RGB12: WS2812B, LED_SMD:LED_WS2812B_PLCC4_5.0x5.0mm_P3.2mm, B.Cu at (302.9, 2.13)
- added RGB13: WS2812B, LED_SMD:LED_WS2812B_PLCC4_5.0x5.0mm_P3.2mm, B.Cu at (177.8, 138.9)
- added RGB14: WS2812B, LED_SMD:LED_WS2812B_PLCC4_5.0x5.0mm_P3.2mm, B.Cu at (228.3, 7.81)
- added RGB2: WS2812B, LED_SMD:LED_WS2812B_PLCC4_5.0x5.0mm_P3.2mm, B.Cu at (284.4, 153.8)
- added RGB3: WS2812B, LED_SMD:LED_WS2812B_PLCC4_5.0x5.0mm_P3.2mm, B.Cu at (75.4, 27.8)
- added RGB4: WS2812B, LED_SMD:LED_WS2812B_PLCC4_5.0x5.0mm_P3.2mm, B.Cu at (358.3, 152.0)
- added RGB5: WS2812B, LED_SMD:LED_WS2812B_PLCC4_5.0x5.0mm_P3.2mm, B.Cu at (32.5, 43.3)
- added RGB6: WS2812B, LED_SMD:LED_WS2812B_PLCC4_5.0x5.0mm_P3.2mm, B.Cu at (384.8, 104.8)
- added RGB7: WS2812B, LED_SMD:LED_WS2812B_PLCC4_5.0x5.0mm_P3.2mm, B.Cu at (32.2, 74.8)
- added RGB8: WS2812B, LED_SMD:LED_WS2812B_PLCC4_5.0x5.0mm_P3.2mm, B.Cu at (386.1, 50.5)
- added RGB9: WS2812B, LED_SMD:LED_WS2812B_PLCC4_5.0x5.0mm_P3.2mm, B.Cu at (30.3, 120.9)
- C1, C2, C3, C4, C5, C6, C7, C8, C9: footprint Capacitors_SMD:C_0805_HandSoldering -> Capacitor_SMD:C_0805_2012Metric_Pad1.18x1.45mm_HandSolder
Connections:
- U2 pad 36: /PF7 -> RGB
Routing:
- net GND: track 109.9 -> 515.7 mm, vias 16 -> 19
- net +5V: track 187.2 -> 575.3 mm, vias 7 -> 12
- net Net-(RGB11-Pad2): track 0.00 -> 110.7 mm
- net Net-(RGB1-Pad2): track 0.00 -> 54.5 mm
- net Net-(RGB3-Pad2): track 0.00 -> 50.6 mm
- net /PF7: track 45.1 -> 0.00 mm, vias 1 -> 0
- net Net-(RGB11-Pad4): track 0.00 -> 43.9 mm
- net Net-(RGB7-Pad2): track 0.00 -> 42.3 mm, vias 0 -> 2
- net RGB: track 0.00 -> 37.8 mm, vias 0 -> 2
- net Net-(RGB5-Pad2): track 0.00 -> 28.1 mm, vias 0 -> 2
- net Net-(R7-Pad2): track 0.00 -> 3.03 mm
- net /col1: track 185.8 -> 184.9 mm
- net /col2: track 196.6 -> 195.8 mm
- net /col0: track 228.2 -> 227.5 mm

Commit message: Add RGB
Finish RGB
Parts:
- moved RGB4 126.5 mm to (234.2, 127.4), turned to 192 degrees
- moved C18 113.5 mm to (238.9, 126.2), turned to 282 degrees
- moved RGB2 110.0 mm to (175.4, 138.9), turned to 180 degrees
- moved RGB6 97.0 mm to (289.7, 123.8), turned to 180 degrees
- moved C17 96.4 mm to (180.2, 138.9), turned to 270 degrees
- moved C19 91.8 mm to (294.5, 123.8), turned to 270 degrees
- moved RGB8 81.3 mm to (355.0, 125.6), turned to 180 degrees
- moved RGB10 73.4 mm to (358.6, 80.7), turned to 270 degrees
- moved C20 71.9 mm to (359.6, 125.4), turned to 270 degrees
- moved C21 68.3 mm to (358.5, 75.9)
- moved RGB12 65.2 mm to (360.5, 32.5), turned to 270 degrees
- moved C22 57.4 mm to (360.6, 27.8)
- moved C16 51.0 mm to (132.7, 131.7), turned to 258 degrees
- moved RGB13 50.3 mm to (128.2, 130.5), turned to 168 degrees
- moved C23 33.6 mm to (247.1, 27.7), turned to 90 degrees
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Routing:
- net GND: track 515.7 -> 928.9 mm, vias 19 -> 23
- net +5V: track 575.3 -> 983.9 mm, vias 12 -> 16
- net Net-(RGB12-Pad2): track 0.00 -> 111.9 mm
- net Net-(RGB6-Pad2): track 0.00 -> 62.3 mm
- net Net-(RGB2-Pad2): track 0.00 -> 59.8 mm
- net Net-(RGB4-Pad2): track 0.00 -> 53.9 mm, vias 0 -> 2
- net Net-(RGB11-Pad2): track 110.7 -> 56.8 mm
- net Net-(RGB10-Pad4): track 0.00 -> 49.4 mm, vias 0 -> 2
- net Net-(RGB13-Pad2): track 0.00 -> 46.9 mm, vias 0 -> 2
- net Net-(RGB10-Pad2): track 0.00 -> 46.0 mm, vias 0 -> 2
- net /row4: track 583.1 -> 581.1 mm
- net /MISO: track 270.6 -> 271.8 mm
